Commit message: Refactor tactile frame definitions and update joint command handling
- Modified tactile_frames.xacro to accept a 'side' parameter, allowing for left and right hand configurations with specific origin and rotation values for tactile sensors.
- Updated README.md to reflect changes in joint command topics, now using percentages for joint positions instead of radians, and added instructions for visualizing tactile data in RViz.
- Adjusted bridge_node.py to handle joint commands as opening percentages, ensuring proper conversion to radians for internal processing.
- Enhanced hand_mapping.py with a new method to convert opening percentages to radians, accommodating the varying upper limits of joints.
- Updated tactile.py to include optional physical pad footprint sizes derived from configuration files, improving tactile region accuracy.
- Modified tactile_cloud_node.py to utilize real pad dimensions for generating tactile point clouds, enhancing spatial accuracy.
- Revised launch file to support optional RViz visualization and tactile cloud generation, improving usability for developers.
- Created RViz configuration files for both left and right hands, facilitating immediate visualization of the robot's tactile feedback.
- Adjusted open_hand.py script to set joint angles correctly in the new percentage-based command system.

File: rh56dftp_description/urdf/rh56dftp.xacro (robot description, xacro)
@@ -32,4 +32,4 @@
   <!-- ================= INSTANTIATE HAND + TACTILE SKIN ================= -->
   <xacro:rh56dftp_hand side="${side_s}" prefix="${prefix_p}"/>
-  <xacro:rh56dftp_tactile_frames prefix="${prefix_p}"/>
+  <xacro:rh56dftp_tactile_frames prefix="${prefix_p}" side="${side_s}"/>
 </robot>

File: rh56dftp_description/urdf/rh56dftp_left.urdf (robot description, URDF)
Before this commit: robot rh56dftp_left, 55 links, 54 joints
Joints:
- joint left_index_palm_touch_joint: origin xyz=0 0 0 rpy=0 0 0 -> xyz=0.009346 0.01361 -0.005947 rpy=1.60167 -0.002672 1.38726
- joint left_index_tip_touch_joint: origin xyz=0 0 0 rpy=0 0 0 -> xyz=-0.00113 -2e-06 -0.000481 rpy=-0.267417 -0.000505 1.57457
- joint left_index_top_touch_joint: origin xyz=0 0 0 rpy=0 0 0 -> xyz=0.01281 0.028816 -0.005389 rpy=1.60342 -0.002735 1.27581
- joint left_little_palm_touch_joint: origin xyz=0 0 0 rpy=0 0 0 -> xyz=0.009383 0.013453 -0.005911 rpy=1.58054 -0.002672 1.38726
- joint left_little_tip_touch_joint: origin xyz=0 0 0 rpy=0 0 0 -> xyz=-0.000812 2.4e-05 -0.000398 rpy=0.255094 -0.004 -1.5708
- joint left_little_top_touch_joint: origin xyz=0 0 0 rpy=0 0 0 -> xyz=0.009995 0.021982 -0.005127 rpy=1.58072 -0.001387 1.27055
- joint left_middle_palm_touch_joint: origin xyz=0 0 0 rpy=0 0 0 -> xyz=0.009387 0.013617 -0.005896 rpy=1.59643 -0.002672 1.38726
- joint left_middle_tip_touch_joint: origin xyz=0 0 0 rpy=0 0 0 -> xyz=-0.000786 -6e-06 -0.000433 rpy=-0.321407 0.004647 1.58354
- joint left_middle_top_touch_joint: origin xyz=0 0 0 rpy=0 0 0 -> xyz=0.014045 0.031523 -0.005277 rpy=1.59534 0.002946 1.26895
- joint left_palm_touch_joint: origin xyz=0 0 0 rpy=0 0 0 -> xyz=0.00018 -0.006891 9.4e-05 rpy=0.14087 0.035477 2.73397
- joint left_ring_palm_touch_joint: origin xyz=0 0 0 rpy=0 0 0 -> xyz=0.009466 0.013563 -0.005878 rpy=1.58851 -0.002672 1.38726
- joint left_ring_tip_touch_joint: origin xyz=0 0 0 rpy=0 0 0 -> xyz=-0.00113 -2e-06 -0.000481 rpy=-0.267417 -0.000505 1.57457
- joint left_ring_top_touch_joint: origin xyz=0 0 0 rpy=0 0 0 -> xyz=0.012935 0.029408 -0.005459 rpy=1.58966 -0.002735 1.27581
- joint left_thumb_middle_touch_joint: origin xyz=0 0 0 rpy=0 0 0 -> xyz=0.011762 0.006056 0.013736 rpy=-0.109716 -0.006889 0.947256
- joint left_thumb_palm_touch_joint: origin xyz=0 0 0 rpy=0 0 0 -> xyz=0.016579 0.028298 0.014575 rpy=-0.030962 -0.007901 0.658301
- joint left_thumb_tip_touch_joint: origin xyz=0 0 0 rpy=0 0 0 -> xyz=1e-05 -0.002125 -0.00081 rpy=0.026243 0.37045 -1.53966
- joint left_thumb_top_touch_joint: origin xyz=0 0 0 rpy=0 0 0 -> xyz=0.006829 0.009674 0.010979 rpy=-0.105254 0.01018 0.928269

File: rh56dftp_description/urdf/rh56dftp_right.urdf (robot description, URDF)
Before this commit: robot rh56dftp_right, 55 links, 54 joints
Joints:
- joint right_index_palm_touch_joint: origin xyz=0 0 0 rpy=0 0 0 -> xyz=0.009283 0.013622 0.005973 rpy=1.54377 -0.000618 1.38857
- joint right_index_tip_touch_joint: origin xyz=0 0 0 rpy=0 0 0 -> xyz=-0.001136 7e-06 -0.000484 rpy=0.266714 -0.000761 -1.5735
- joint right_index_top_touch_joint: origin xyz=0 0 0 rpy=0 0 0 -> xyz=0.012839 0.02888 0.005474 rpy=1.54129 0.002237 1.27695
- joint right_little_palm_touch_joint: origin xyz=0 0 0 rpy=0 0 0 -> xyz=0.009354 0.013454 0.005832 rpy=1.55918 -0.000618 1.38857
- joint right_little_tip_touch_joint: origin xyz=0 0 0 rpy=0 0 0 -> xyz=-0.000811 1.2e-05 -0.000398 rpy=-0.256934 -0.000876 1.56988
- joint right_little_top_touch_joint: origin xyz=0 0 0 rpy=0 0 0 -> xyz=0.009976 0.021938 -0.004987 rpy=1.55905 -0.001387 1.27055
- joint right_middle_palm_touch_joint: origin xyz=0 0 0 rpy=0 0 0 -> xyz=0.009329 0.013585 0.005847 rpy=1.54377 -0.000618 1.38857
- joint right_middle_tip_touch_joint: origin xyz=0 0 0 rpy=0 0 0 -> xyz=-0.000783 -1.2e-05 -0.000434 rpy=-0.322021 0.001984 1.58258
- joint right_middle_top_touch_joint: origin xyz=0 0 0 rpy=0 0 0 -> xyz=0.014176 0.031963 0.005275 rpy=1.54456 -0.004895 1.27136
- joint right_palm_touch_joint: origin xyz=0 0 0 rpy=0 0 0 -> xyz=-0.000774 -0.007075 4e-05 rpy=-0.140338 0.031573 0.400942
- joint right_ring_palm_touch_joint: origin xyz=0 0 0 rpy=0 0 0 -> xyz=0.009295 0.013631 0.005825 rpy=1.54895 -0.000618 1.38857
- joint right_ring_tip_touch_joint: origin xyz=0 0 0 rpy=0 0 0 -> xyz=-0.001136 7e-06 -0.000484 rpy=0.266714 -0.000761 -1.5735
- joint right_ring_top_touch_joint: origin xyz=0 0 0 rpy=0 0 0 -> xyz=0.012939 0.029407 0.005466 rpy=1.54669 0.002237 1.27695
- joint right_thumb_middle_touch_joint: origin xyz=0 0 0 rpy=0 0 0 -> xyz=-0.011522 0.006102 0.013701 rpy=0.109631 -0.020842 2.18981
- joint right_thumb_palm_touch_joint: origin xyz=0 0 0 rpy=0 0 0 -> xyz=-0.016374 0.028338 0.014539 rpy=0.031405 -0.006998 2.48191
- joint right_thumb_tip_touch_joint: origin xyz=0 0 0 rpy=0 0 0 -> xyz=-4e-06 0.002134 -0.000813 rpy=0.007998 0.371429 1.56075
- joint right_thumb_top_touch_joint: origin xyz=0 0 0 rpy=0 0 0 -> xyz=-0.00672 0.009818 0.010921 rpy=0.104105 0.004501 2.21398

File: rh56dftp_description/urdf/tactile_frames.xacro (robot description, xacro)
@@ -2,5 +2,5 @@
 <!-- GENERATED by tools/build.py from tactile/tactile_layout.yaml — DO NOT EDIT BY HAND -->
 <robot xmlns:xacro="http://www.ros.org/wiki/xacro">
-  <xacro:macro name="rh56dftp_tactile_frames" params="prefix">
+  <xacro:macro name="rh56dftp_tactile_frames" params="prefix side">
     <!-- little_tip: dds=fingerone_tip_touch grid=3x3 (9 taxels) modbus=3000 -->
     <link name="${prefix}little_tip_touch"/>
@@ -8,5 +8,6 @@
       <parent link="${prefix}little_tip"/>
       <child link="${prefix}little_tip_touch"/>
-      <origin xyz="0 0 0" rpy="0 0 0"/>
+      <xacro:if value="${side == 'left'}"><origin xyz="-0.000812 2.4e-05 -0.000398" rpy="0.255094 -0.004 -1.5708"/></xacro:if>
+      <xacro:if value="${side == 'right'}"><origin xyz="-0.000811 1.2e-05 -0.000398" rpy="-0.256934 -0.000876 1.56988"/></xacro:if>
     </joint>
     <!-- little_top: dds=fingerone_top_touch grid=12x8 (96 taxels) modbus=3018 -->
@@ -15,5 +16,6 @@
       <parent link="${prefix}little_2"/>
       <child link="${prefix}little_top_touch"/>
-      <origin xyz="0 0 0" rpy="0 0 0"/>
+      <xacro:if value="${side == 'left'}"><origin xyz="0.009995 0.021982 -0.005127" rpy="1.58072 -0.001387 1.27055"/></xacro:if>
+      <xacro:if value="${side == 'right'}"><origin xyz="0.009976 0.021938 -0.004987" rpy="1.55905 -0.001387 1.27055"/></xacro:if>
     </joint>
     <!-- little_palm: dds=fingerone_palm_touch grid=10x8 (80 taxels) modbus=3210 -->
@@ -22,5 +24,6 @@
       <parent link="${prefix}little_1"/>
       <child link="${prefix}little_palm_touch"/>
-      <origin xyz="0 0 0" rpy="0 0 0"/>
+      <xacro:if value="${side == 'left'}"><origin xyz="0.009383 0.013453 -0.005911" rpy="1.58054 -0.002672 1.38726"/></xacro:if>
+      <xacro:if value="${side == 'right'}"><origin xyz="0.009354 0.013454 0.005832" rpy="1.55918 -0.000618 1.38857"/></xacro:if>
     </joint>
     <!-- ring_tip: dds=fingertwo_tip_touch grid=3x3 (9 taxels) modbus=3370 -->
@@ -29,5 +32,6 @@
       <parent link="${prefix}ring_tip"/>
       <child link="${prefix}ring_tip_touch"/>
-      <origin xyz="0 0 0" rpy="0 0 0"/>
+      <xacro:if value="${side == 'left'}"><origin xyz="-0.00113 -2e-06 -0.000481" rpy="-0.267417 -0.000505 1.57457"/></xacro:if>
+      <xacro:if value="${side == 'right'}"><origin xyz="-0.001136 7e-06 -0.000484" rpy="0.266714 -0.000761 -1.5735"/></xacro:if>
     </joint>
     <!-- ring_top: dds=fingertwo_top_touch grid=12x8 (96 taxels) modbus=3388 -->
@@ -36,5 +40,6 @@
       <parent link="${prefix}ring_2"/>
       <child link="${prefix}ring_top_touch"/>
-      <origin xyz="0 0 0" rpy="0 0 0"/>
+      <xacro:if value="${side == 'left'}"><origin xyz="0.012935 0.029408 -0.005459" rpy="1.58966 -0.002735 1.27581"/></xacro:if>
+      <xacro:if value="${side == 'right'}"><origin xyz="0.012939 0.029407 0.005466" rpy="1.54669 0.002237 1.27695"/></xacro:if>
     </joint>
     <!-- ring_palm: dds=fingertwo_palm_touch grid=10x8 (80 taxels) modbus=3580 -->
@@ -43,5 +48,6 @@
       <parent link="${prefix}ring_1"/>
       <child link="${prefix}ring_palm_touch"/>
-      <origin xyz="0 0 0" rpy="0 0 0"/>
+      <xacro:if value="${side == 'left'}"><origin xyz="0.009466 0.013563 -0.005878" rpy="1.58851 -0.002672 1.38726"/></xacro:if>
+      <xacro:if value="${side == 'right'}"><origin xyz="0.009295 0.013631 0.005825" rpy="1.54895 -0.000618 1.38857"/></xacro:if>
     </joint>
     <!-- middle_tip: dds=fingerthree_tip_touch grid=3x3 (9 taxels) modbus=3740 -->
@@ -50,5 +56,6 @@
       <parent link="${prefix}middle_tip"/>
       <child link="${prefix}middle_tip_touch"/>
-      <origin xyz="0 0 0" rpy="0 0 0"/>
+      <xacro:if value="${side == 'left'}"><origin xyz="-0.000786 -6e-06 -0.000433" rpy="-0.321407 0.004647 1.58354"/></xacro:if>
+      <xacro:if value="${side == 'right'}"><origin xyz="-0.000783 -1.2e-05 -0.000434" rpy="-0.322021 0.001984 1.58258"/></xacro:if>
     </joint>
     <!-- middle_top: dds=fingerthree_top_touch grid=12x8 (96 taxels) modbus=3758 -->
@@ -57,5 +64,6 @@
       <parent link="${prefix}middle_2"/>
       <child link="${prefix}middle_top_touch"/>
-      <origin xyz="0 0 0" rpy="0 0 0"/>
+      <xacro:if value="${side == 'left'}"><origin xyz="0.014045 0.031523 -0.005277" rpy="1.59534 0.002946 1.26895"/></xacro:if>
+      <xacro:if value="${side == 'right'}"><origin xyz="0.014176 0.031963 0.005275" rpy="1.54456 -0.004895 1.27136"/></xacro:if>
     </joint>
     <!-- middle_palm: dds=fingerthree_palm_touch grid=10x8 (80 taxels) modbus=3950 -->
@@ -64,5 +72,6 @@
       <parent link="${prefix}middle_1"/>
       <child link="${prefix}middle_palm_touch"/>
-      <origin xyz="0 0 0" rpy="0 0 0"/>
+      <xacro:if value="${side == 'left'}"><origin xyz="0.009387 0.013617 -0.005896" rpy="1.59643 -0.002672 1.38726"/></xacro:if>
+      <xacro:if value="${side == 'right'}"><origin xyz="0.009329 0.013585 0.005847" rpy="1.54377 -0.000618 1.38857"/></xacro:if>
     </joint>
     <!-- index_tip: dds=fingerfour_tip_touch grid=3x3 (9 taxels) modbus=4110 -->
@@ -71,5 +80,6 @@
       <parent link="${prefix}index_tip"/>
       <child link="${prefix}index_tip_touch"/>
-      <origin xyz="0 0 0" rpy="0 0 0"/>
+      <xacro:if value="${side == 'left'}"><origin xyz="-0.00113 -2e-06 -0.000481" rpy="-0.267417 -0.000505 1.57457"/></xacro:if>
+      <xacro:if value="${side == 'right'}"><origin xyz="-0.001136 7e-06 -0.000484" rpy="0.266714 -0.000761 -1.5735"/></xacro:if>
     </joint>
     <!-- index_top: dds=fingerfour_top_touch grid=12x8 (96 taxels) modbus=4128 -->
@@ -78,5 +88,6 @@
       <parent link="${prefix}index_2"/>
       <child link="${prefix}index_top_touch"/>
-      <origin xyz="0 0 0" rpy="0 0 0"/>
+      <xacro:if value="${side == 'left'}"><origin xyz="0.01281 0.028816 -0.005389" rpy="1.60342 -0.002735 1.27581"/></xacro:if>
+      <xacro:if value="${side == 'right'}"><origin xyz="0.012839 0.02888 0.005474" rpy="1.54129 0.002237 1.27695"/></xacro:if>
     </joint>
     <!-- index_palm: dds=fingerfour_palm_touch grid=10x8 (80 taxels) modbus=4320 -->
@@ -85,5 +96,6 @@
       <parent link="${prefix}index_1"/>
       <child link="${prefix}index_palm_touch"/>
-      <origin xyz="0 0 0" rpy="0 0 0"/>
+      <xacro:if value="${side == 'left'}"><origin xyz="0.009346 0.01361 -0.005947" rpy="1.60167 -0.002672 1.38726"/></xacro:if>
+      <xacro:if value="${side == 'right'}"><origin xyz="0.009283 0.013622 0.005973" rpy="1.54377 -0.000618 1.38857"/></xacro:if>
     </joint>
     <!-- thumb_tip: dds=fingerfive_tip_touch grid=3x3 (9 taxels) modbus=4480 -->
@@ -92,5 +104,6 @@
       <parent link="${prefix}thumb_tip"/>
       <child link="${prefix}thumb_tip_touch"/>
-      <origin xyz="0 0 0" rpy="0 0 0"/>
+      <xacro:if value="${side == 'left'}"><origin xyz="1e-05 -0.002125 -0.00081" rpy="0.026243 0.37045 -1.53966"/></xacro:if>
+      <xacro:if value="${side == 'right'}"><origin xyz="-4e-06 0.002134 -0.000813" rpy="0.007998 0.371429 1.56075"/></xacro:if>
     </joint>
     <!-- thumb_top: dds=fingerfive_top_touch grid=12x8 (96 taxels) modbus=4498 -->
@@ -99,5 +112,6 @@
       <parent link="${prefix}thumb_4"/>
       <child link="${prefix}thumb_top_touch"/>
-      <origin xyz="0 0 0" rpy="0 0 0"/>
+      <xacro:if value="${side == 'left'}"><origin xyz="0.006829 0.009674 0.010979" rpy="-0.105254 0.01018 0.928269"/></xacro:if>
+      <xacro:if value="${side == 'right'}"><origin xyz="-0.00672 0.009818 0.010921" rpy="0.104105 0.004501 2.21398"/></xacro:if>
     </joint>
     <!-- thumb_middle: dds=fingerfive_middle_touch grid=3x3 (9 taxels) modbus=4690 -->
@@ -106,5 +120,6 @@
       <parent link="${prefix}thumb_3"/>
       <child link="${prefix}thumb_middle_touch"/>
-      <origin xyz="0 0 0" rpy="0 0 0"/>
+      <xacro:if value="${side == 'left'}"><origin xyz="0.011762 0.006056 0.013736" rpy="-0.109716 -0.006889 0.947256"/></xacro:if>
+      <xacro:if value="${side == 'right'}"><origin xyz="-0.011522 0.006102 0.013701" rpy="0.109631 -0.020842 2.18981"/></xacro:if>
     </joint>
     <!-- thumb_palm: dds=fingerfive_palm_touch grid=12x8 (96 taxels) modbus=4708 -->
@@ -113,5 +128,6 @@
       <parent link="${prefix}thumb_2"/>
       <child link="${prefix}thumb_palm_touch"/>
-      <origin xyz="0 0 0" rpy="0 0 0"/>
+      <xacro:if value="${side == 'left'}"><origin xyz="0.016579 0.028298 0.014575" rpy="-0.030962 -0.007901 0.658301"/></xacro:if>
+      <xacro:if value="${side == 'right'}"><origin xyz="-0.016374 0.028338 0.014539" rpy="0.031405 -0.006998 2.48191"/></xacro:if>
     </joint>
     <!-- palm: dds=palm_touch grid=14x8 (112 taxels) modbus=4900 -->
@@ -120,5 +136,6 @@
       <parent link="${prefix}palm"/>
       <child link="${prefix}palm_touch"/>
-      <origin xyz="0 0 0" rpy="0 0 0"/>
+      <xacro:if value="${side == 'left'}"><origin xyz="0.00018 -0.006891 9.4e-05" rpy="0.14087 0.035477 2.73397"/></xacro:if>
+      <xacro:if value="${side == 'right'}"><origin xyz="-0.000774 -0.007075 4e-05" rpy="-0.140338 0.031573 0.400942"/></xacro:if>
     </joint>
   </xacro:macro>
